File: electronics/kicad/LedCube/LedCube.kicad_pcb (KiCad board)
At the start: 2 copper layers, 20 parts, among them J1 Conn_01x03, J2 Conn_01x03, J3 Conn_01x03, J4 Conn_01x04, J5 COM, J6 Conn_01x02, J7 JTAG, U1 ESP32

Commit message: Add esp32 devkit footprint
Parts:
- added U2: ESP32-DevKitC, Esp32:ESP32-DevKitC, F.Cu at (60.1, 72.8)
- U1: value ESP32 -> ESP32-S3-DevKitC; footprint Esp32:ESP32-DevKitC -> Espressif:ESP32-S3-DevKitC
- moved U1 37.1 mm to (24.1, 60.2)
Connections:
- U1 pad 1: Net-(U1-Pad1) -> +3V3
- U1 pad 2: unconnected-(U1-Pad2) -> +3V3
- U1 pad 22: unconnected-(U1-Pad22) -> GND
- U1 pad 23: unconnected-(U1-Pad23) -> GND
- U1 pad 24: unconnected-(U1-Pad24) -> GND
- U1 pad 3: Net-(U1-Pad3) -> unconnected-(U1-CHIP_PU-Pad3)
- U1 pad 4: Net-(U1-Pad3) -> unconnected-(U1-GPIO4/ADC1_CH3-Pad4)

Commit message: Finish KiCad PCB board
Parts:
- removed U1: ESP32-S3-DevKitC, Espressif:ESP32-S3-DevKitC
- removed U2: ESP32-DevKitC, Esp32:ESP32-DevKitC
- added C2: 100uF, Capacitor_THT:C_Radial_D5.0mm_H5.0mm_P2.00mm, F.Cu at (135.2, 116.5)
- added H1: MountingHole, MountingHole:MountingHole_3.2mm_M3_Pad, F.Cu at (117.2, 80.0)
- added H2: MountingHole, MountingHole:MountingHole_3.2mm_M3_Pad, F.Cu at (193.2, 80.0)
- added H3: MountingHole, MountingHole:MountingHole_3.2mm_M3_Pad, F.Cu at (193.2, 116.0)
- added H4: MountingHole, MountingHole:MountingHole_3.2mm_M3_Pad, F.Cu at (117.2, 116.0)
- added U3: ESP32-DevKitM, Espressif:ESP32-DevKitM, F.Cu at (147.3, 104.7)
- C1: value 220uF -> 100uF; footprint Capacitor_THT:C_Radial_D6.3mm_H5.0mm_P2.50mm -> Capacitor_THT:C_Radial_D5.0mm_H5.0mm_P2.00mm
- J5: footprint Connector_PinHeader_1.27mm:PinHeader_2x03_P1.27mm_Vertical -> Connectors:ESP_PROG_COM
- J6: footprint Connector_JST:JST_XH_B2B-XH-AM_1x02_P2.50mm_Vertical -> Connector_JST:JST_XH_B2B-XH-A_1x02_P2.50mm_Vertical
- J7: footprint Connector_PinHeader_1.27mm:PinHeader_2x05_P1.27mm_Vertical -> Connectors:ESP_PROG_JTAG
- moved D1 48.2 mm to (178.5, 108.3), turned to -90 degrees
- moved J5 48.2 mm to (194.0, 92.3), turned to 180 degrees
- moved J6 44.8 mm to (183.8, 116.0)
- moved C1 40.9 mm to (185.8, 108.5)
- moved R9 38.4 mm to (171.7, 111.2), turned to -90 degrees
- moved J7 37.4 mm to (194.0, 106.8), turned to 180 degrees
- moved G*** 31.9 mm to (130.5, 89.0)
- moved R7 28.3 mm to (166.7, 111.2), turned to -90 degrees
- moved J2 27.2 mm to (154.8, 116.0)
- moved J3 25.4 mm to (166.7, 116.0)
- moved R6 21.8 mm to (159.8, 111.2), turned to -90 degrees
- moved J1 17.8 mm to (142.8, 116.0)
- moved J4 17.1 mm to (130.5, 116.8), turned to -90 degrees
- moved R8 16.5 mm to (169.2, 111.2), turned to -90 degrees
- moved R5 10.5 mm to (157.2, 111.2), turned to -90 degrees
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Routing:
- net +3V3: track 0.00 -> 90.0 mm
- net UART1_RX: track 0.00 -> 62.7 mm
- net UART1_TX: track 0.00 -> 62.5 mm
- net UART0_TX: track 0.00 -> 58.7 mm
- net UART0_RX: track 0.00 -> 50.8 mm
- net D3: track 0.00 -> 47.2 mm
- net D2: track 0.00 -> 40.1 mm
- net D1: track 0.00 -> 38.6 mm
- net D0: track 0.00 -> 37.2 mm
- net RESET: track 0.00 -> 37.1 mm
- net TCK: track 0.00 -> 30.6 mm, vias 0 -> 1
- net TDI: track 0.00 -> 29.5 mm
- net TDO: track 0.00 -> 29.5 mm, vias 0 -> 1
- net GPIO_0: track 0.00 -> 20.5 mm
- net D4: track 0.00 -> 18.1 mm
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- added copper zone on B.Cu, net GND
- added copper zone on F.Cu, net GND
Other:
- board outline added: 86 x 46 mm
- board text added: "+"
- board text added: "-"
- board text added: "0"
- board text added: "1"
- board text added: "2"
- board text added: "3"
- board text added: "4"
- board text added: "5"
- board text added: "5v"
- board text added: "6"
- board text added: "7"
- board text added: "8"
- board text added: "COM"
- board text added: "Display"
- board text added: "JTAG"
- board text added: "Led Data Pins"
